File: hardware/leadtech-arduino-CSPG_concept.sch (EAGLE design)
At the start: 18 parts, among them J1 CON_HEADER_1X08-PTH, J2 CON_HEADER_1X08-PTH, J3 CON_HEADER_1X08-PTH, J4 CON_HEADER_1X06-PTH, J5 CON_HEADER_1X05-PTH, J6 CON_HEADER_1X02-PTH, J7 CON_HEADER_1X05-PTH, J8 CON_HEADER_1X08-PTH, P1 CON_HEADER_2X09, P2 CON_HEADER_2X09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

Commit message: update on schematic, placed voltage level shift buffer for RF-ID I/O
Parts:
- removed R3: 3.6K, dp_devices.v6:RESISTOR-0603
- removed R4: 6.8K, dp_devices.v6:RESISTOR-0603
- added C1: 0.1uF, dp_devices.v6:CAPACITOR_NPOL-PTH_0.1"
- added IC1: CD4050B, 40xx:4050N
- R5: value 3.6K -> 4.7K
Connections:
- removed net ARDUINO-11: J1.4, J8.3
- removed net ARDUINO-13: J1.6, J8.2
- new net N$2: IC1A.O, J8.1
- new net N$3: IC1B.I, J1.6
- new net N$4: IC1B.O, J8.2
- new net N$5: IC1C.I, J1.4
- new net N$6: IC1C.O, J8.3
- new net N$7: IC1D.O, J8.7
- net ARDUINO-10: now also IC1A.I; no longer J8.1
- net ARDUINO-9: now also IC1D.I; no longer J8.7
- net GND: now also C1.2, IC1P.VSS
- net N$1: now also C1.1, IC1P.VDD
Other:
- note removed: "OLED RES -> 22 DC -> 24 CS -> 26"
- note removed: "RF-ID SS/SDA -> 10 RST -> 9"
- moved on the sheet: J1, J2, J3, J4, J7, J8, LED1, P1, P2, R1, R2, R5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
